Commit message: cartesian failed sometimes

File: src/robo_arm6/urdf/robo_arm6.urdf (robot description, URDF)
Before this commit: robot robo_arm6, 7 links, 6 joints
Joints:
- joint joint2: limit lower=0 upper=3.14 effort=0 velocity=0 -> lower=-3.14 upper=3.14 effort=0 velocity=0; origin xyz=-0.0557 0 0.063 rpy=0 -1.5376 0 -> xyz=-0.0557 0 0.063 rpy=-1.57 0 1.57
- joint joint3: origin xyz=0.38 0 -0.01983 rpy=0 0 0 -> xyz=0.38 0 -0.01983 rpy=0 0 3.14
- joint joint5: limit lower=-1.57 upper=4.71 effort=0 velocity=0 -> lower=0 upper=6.28 effort=0 velocity=0; origin xyz=0 -0.031 0.1572 rpy=-1.5708 0 0 -> xyz=0 -0.031 0.1572 rpy=-1.5708 1.5708 0
