Commit message: feat: rewrite gravity compensation with RNEA and add test infrastructure
- Regenerate gravity_comp.c using RNEA-based approach for correctness
- Add generate_gravity_comp_rnea.py generator script
- Add test_gravity_comp and gravity_comp_debug nodes
- Add launch files for gravity comp testing/debugging
- Use full-precision rpy values in URDF
- Fix .position.z() -> .position.z bug in real_world_new.cpp
- Reduce gravity closure log verbosity (INFO -> DEBUG)

Co-Authored-By: Claude Opus 4.6 <noreply@anthropic.com>

File: src/robo_arm6/urdf/robo_arm6.urdf (robot description, URDF)
Before this commit: robot robo_arm6, 7 links, 6 joints
Joints:
- joint joint2: origin xyz=-0.0557 0 0.063 rpy=-1.57 0 1.57 -> xyz=-0.0557 0 0.063 rpy=-1.5707963267948966 0 1.5707963267948966
- joint joint3: origin xyz=0.38 0 -0.01983 rpy=0 0 3.14 -> xyz=0.38 0 -0.01983 rpy=0 0 3.141592653589793
- joint joint4: origin xyz=0.054993 -0.15447 -0.039 rpy=1.5708 0 0 -> xyz=0.054993 -0.15447 -0.039 rpy=1.5707963267948966 0 0
- joint joint5: origin xyz=0 -0.031 0.1572 rpy=-1.5708 1.5708 0 -> xyz=0 -0.031 0.1572 rpy=-1.5707963267948966 1.5707963267948966 0
- joint joint6: origin xyz=0.096475 0 0.032 rpy=0 1.5708 0 -> xyz=0.096475 0 0.032 rpy=0 1.5707963267948966 0
