Commit message: change receive_data function from executor run and wait in while loop to timer callback

File: src/arms/robo_arm10/urdf/robo_arm10.urdf (robot description, URDF)
Before this commit: robot robo_arm10, 8 links, 7 joints
Joints:
- joint joint1: limit lower=-2.00713 upper=0.61087 effort=0 velocity=0 -> lower=-2.00713 upper=0.9 effort=0 velocity=0
- joint joint3: limit lower=-1.27409 upper=1.27409 effort=0 velocity=0 -> lower=-1.5 upper=1.5 effort=0 velocity=0
- joint joint4: limit lower=0 upper=6.2832 effort=0 velocity=0 -> lower=-6.2832 upper=0 effort=0 velocity=0
- joint joint5: limit lower=-1.74533 upper=1.74533 effort=0 velocity=0 -> lower=4.2 upper=8.4 effort=0 velocity=0
- joint joint6: limit lower=-3.1416 upper=3.1416 effort=0 velocity=0 -> lower=-3.3 upper=3.3 effort=0 velocity=0

Commit message: 添加了pyroki节点作为teleop

File: src/arms/robo_arm10/urdf/robo_arm10.urdf (robot description, URDF)
Before this commit: robot robo_arm10, 8 links, 7 joints
Joints:
- joint joint1: limit lower=-2.00713 upper=0.9 effort=0 velocity=0 -> lower=-2.5 upper=1.5 effort=0 velocity=0
- joint joint2: limit lower=-2.84489 upper=0 effort=0 velocity=0 -> lower=-3.3 upper=0.5 effort=0 velocity=0
- joint joint3: limit lower=-1.5 upper=1.5 effort=0 velocity=0 -> lower=-2.0 upper=2.0 effort=0 velocity=0
- joint joint4: limit lower=-6.2832 upper=0 effort=0 velocity=0 -> lower=-6.8 upper=0.5 effort=0 velocity=0
- joint joint5: limit lower=4.2 upper=8.4 effort=0 velocity=0 -> lower=3.7 upper=8.9 effort=0 velocity=0
- joint joint6: limit lower=-3.3 upper=3.3 effort=0 velocity=0 -> lower=-3.8 upper=3.8 effort=0 velocity=0

Commit message: may16 update readme, add use sim time in pyroki.launch.py, add gripper joint in srdf10

File: src/arms/robo_arm10/urdf/robo_arm10.urdf (robot description, URDF)
Before this commit: robot robo_arm10, 8 links, 7 joints
Links:
- link base_link: mass 0.0190299341581886 -> None

Commit message: may27

File: src/arms/robo_arm10/urdf/robo_arm10.urdf (robot description, URDF)
Before this commit: robot robo_arm10, 8 links, 7 joints
Joints:
- joint joint1: limit lower=-2.5 upper=1.5 effort=0 velocity=0 -> lower=-6.28 upper=6.28 effort=0 velocity=0
- joint joint2: limit lower=-3.3 upper=0.5 effort=0 velocity=0 -> lower=-6.28 upper=6.28 effort=0 velocity=0
- joint joint3: limit lower=-2.0 upper=2.0 effort=0 velocity=0 -> lower=-6.28 upper=6.28 effort=0 velocity=0
- joint joint4: limit lower=-6.8 upper=0.5 effort=0 velocity=0 -> lower=-6.28 upper=6.28 effort=0 velocity=0
- joint joint5: limit lower=3.7 upper=8.9 effort=0 velocity=0 -> lower=-6.28 upper=6.28 effort=0 velocity=0
- joint joint6: limit lower=-3.8 upper=3.8 effort=0 velocity=0 -> lower=-6.28 upper=6.28 effort=0 velocity=0

Commit message: [Log] 28052026 UC backup

File: src/arms/robo_arm10/urdf/robo_arm10.urdf (robot description, URDF)
Before this commit: robot robo_arm10, 8 links, 7 joints
Joints:
- joint joint1: limit lower=-6.28 upper=6.28 effort=0 velocity=0 -> lower=-1.5708 upper=1.5708 effort=0 velocity=0
- joint joint2: limit lower=-6.28 upper=6.28 effort=0 velocity=0 -> lower=-1.5708 upper=0 effort=0 velocity=0
- joint joint3: limit lower=-6.28 upper=6.28 effort=0 velocity=0 -> lower=-1.3416 upper=1.3416 effort=0 velocity=0
- joint joint4: limit lower=-6.28 upper=6.28 effort=0 velocity=0 -> lower=-3.1416 upper=3.1416 effort=0 velocity=0
- joint joint5: limit lower=-6.28 upper=6.28 effort=0 velocity=0 -> lower=-1.5 upper=1.2 effort=0 velocity=0
- joint joint6: limit lower=-6.28 upper=6.28 effort=0 velocity=0 -> lower=-3.1416 upper=3.1416 effort=0 velocity=0

File: src/arms/uc_planning_urdf/urdf/uc_planning_urdf.urdf (robot description, URDF)
Before this commit: robot controller_urdf_v4, 7 links, 6 joints
Links:
- added link gripper
- link base_link: mass 0.437449001710866 -> 0.30266; geometry collision mesh filename=package://uc_planning_urdf/meshes/base_link.STL; visual mesh filename=package://uc_planning_urdf/meshes/base_link.STL
- link link1: mass 0.480839058562563 -> 1.2943; geometry collision mesh filename=package://uc_planning_urdf/meshes/link1.STL; visual mesh filename=package://uc_planning_urdf/meshes/link1.STL
- link link2: mass 0.149564607656572 -> 0.90895; geometry collision mesh filename=package://uc_planning_urdf/meshes/link2.STL; visual mesh filename=package://uc_planning_urdf/meshes/link2.STL
- link link3: mass 0.103129376453745 -> 0.980291734182957; geometry visual mesh filename=package://uc_planning_urdf/meshes/link3.STL
- link link4: mass 0.0799489748689938 -> 0.547610316811054; geometry collision mesh filename=package://uc_planning_urdf/meshes/link4.STL; visual mesh filename=package://uc_planning_urdf/meshes/link4.STL
- link link5: mass 0.195241175955602 -> 0.385427420442394; geometry collision mesh filename=package://uc_planning_urdf/meshes/link5.STL; visual mesh filename=package://uc_planning_urdf/meshes/link5.STL
- link link6: mass 0.009551051850161 -> 1.63806650428865; geometry collision mesh filename=package://uc_planning_urdf/meshes/link6.STL; visual mesh filename=package://uc_planning_urdf/meshes/link6.STL
Joints:
- added joint gripper: type fixed, parent link6, child gripper, origin xyz=-0.019511 -0.00016032 0.16996 rpy=0 -0.79367 0.00072185, axis 0 0 0
- joint joint1: limit lower=-3.14 upper=3.14 effort=0 velocity=0 -> lower=-1.5708 upper=1.5708 effort=0 velocity=0; origin xyz=0 0 0.0426 rpy=0 0 0 -> xyz=0 0 0 rpy=0 0 0
- joint joint2: limit lower=-3.14 upper=3.14 effort=0 velocity=0 -> lower=-1.5708 upper=0 effort=0 velocity=0; origin xyz=0.02 0.055 0.064041 rpy=1.5708 -1.5708 0 -> xyz=0 0.062 0.068 rpy=1.5708 -1.5708 0
- joint joint3: axis 0 0 1 -> 0 0 -1; limit lower=-3.14 upper=3.14 effort=0 velocity=0 -> lower=-1.3416 upper=1.3416 effort=0 velocity=0; origin xyz=0 0.1 0 rpy=0 0 0 -> xyz=0 0.38 0.003 rpy=0 0 0
- joint joint4: limit lower=-3.14 upper=3.14 effort=0 velocity=0 -> lower=-3.1416 upper=3.1416 effort=0 velocity=0; origin xyz=0.1 0 0.055 rpy=-1.5708 0 -1.5708 -> xyz=0.095 0 0.05875 rpy=-1.5708 0 -1.5708
- joint joint5: axis 0 0.018306 -0.99983 -> 0 0 -1; limit lower=-3.14 upper=3.14 effort=0 velocity=0 -> lower=-1.5 upper=1.2 effort=0 velocity=0; origin xyz=5.5833E-05 -0.0030495 0.0501 rpy=1.5708 -1.5708 0 -> xyz=0 0.051 0.1455 rpy=1.5708 -1.5708 0
- joint joint6: axis 0.0036982 0.018306 -0.99983 -> -0.0082726 -0.00012944 0.99997; limit lower=-3.14 upper=3.14 effort=0 velocity=0 -> lower=-3.1416 upper=3.1416 effort=0 velocity=0; origin xyz=0.059944 0.099692 -0.0011752 rpy=1.5708 0 0 -> xyz=0.044798 0.00037066 0.051 rpy=-1.5708 0 -1.5708

Commit message: may30

File: src/arms/robo_arm10/urdf/robo_arm10.urdf (robot description, URDF)
Before this commit: robot robo_arm10, 8 links, 7 joints
Joints:
- joint gripper: origin xyz=0 0 0.15 rpy=0 0 0 -> xyz=0 0 0.1854 rpy=0 0 0

Commit message: feat: 添加了turn模式下的可视化，添加了视觉识别节点marker reco

File: src/arms/robo_arm10/urdf/robo_arm10.urdf (robot description, URDF)
Before this commit: robot robo_arm10, 8 links, 7 joints
Joints:
- joint gripper: origin xyz=0 0 0.1854 rpy=0 0 0 -> xyz=0 0 0.14 rpy=0 0 0
