Commit message: new urdf and workspace visualizer using fibonacci to sample

File: src/arms/robo_arm10/urdf/robo_arm10.urdf (robot description, URDF)
Before this commit: robot robo_arm10, 8 links, 7 joints
Joints:
- joint joint1: limit lower=-1.5708 upper=1.5708 effort=0 velocity=0 -> lower=-2.3562 upper=2.3562 effort=0 velocity=0
- joint joint2: limit lower=-1.5708 upper=0 effort=0 velocity=0 -> lower=-2.8448 upper=-0.29671 effort=0 velocity=0
- joint joint3: limit lower=-1.3416 upper=1.3416 effort=0 velocity=0 -> lower=-1.274 upper=1.047 effort=0 velocity=0
- joint joint5: limit lower=-1.5 upper=1.2 effort=0 velocity=0 -> lower=-1.74533 upper=1.74533 effort=0 velocity=0

File: src/arms/uc_planning_urdf/urdf/uc_planning_urdf.urdf (robot description, URDF)
Before this commit: robot uc_planning_urdf, 8 links, 7 joints
Links:
- link link3: geometry collision mesh filename=package://uc_planning_urdf/meshes/link3.STL; visual mesh filename=package://uc_planning_urdf/meshes/link3.STL
