Commit message: refactor: change to combined URDF and update sampling algorithm

File: src/arms/combine_urdf/urdf/combine_urdf.urdf (robot description, URDF)
Before this commit: robot combine_urdf, 10 links, 9 joints
Joints:
- joint base_joint: origin xyz=0 0.23371 0.088788 rpy=0 0 1.5943 -> xyz=0.23371 0 0.088788 rpy=0 0 0.023499
- joint ground_to_chasis_fixed: origin xyz=1 0.35 0.842 rpy=0 0 1.5707963267949 -> xyz=1 0.35 0.842 rpy=0 0 -3.14159265358979323846

File: src/arms/robo_arm13/urdf/robo_arm13.urdf (robot description, URDF)
Before this commit: robot robo_arm13, 8 links, 7 joints
Joints:
- joint joint2: axis 0 0 1 -> 0 0 -1

Commit message: merge readme.md 2026/8/16

File: src/arms/combine_urdf/urdf/combine_urdf.urdf (robot description, URDF)
Before this commit: robot combine_urdf, 10 links, 9 joints
Links:
- removed link ground
Joints:
- removed joint ground_to_chasis_fixed

Commit message: III type task using improved algorithm

File: src/arms/combine_urdf/urdf/combine_urdf.urdf (robot description, URDF)
Before this commit: robot combine_urdf, 9 links, 8 joints
Links:
- removed link chasis_link
- added link chassis_link, mass 4.54836449313373; collision mesh filename=package://combine_urdf/meshes/chassis_link.STL; visual mesh filename=package://combine_urdf/meshes/chassis_link.STL
Joints:
- joint base_joint: parent chasis_link -> chassis_link
